File: hardware/eagle/rt_solder_simple_V1.2.brd (EAGLE design)
At the start: 71.7 x 59.1 mm, 33 parts, among them IC1 MEGA8-P, IC2 78L05, IC3 TLC27L2ACP, Q1 2N7000, Q3 IRF5305, X1 POWER, X2 Solder

Commit message: part list added
Parts:
- C1: value 4.7µF -> 4.7µF 10V
- C2, C5: value 470µF -> 470µF 16V
- L1: value 22µH -> 22µH or 10R
- Q1: value 2N7000 -> 2N7000 N-CH
- Q3: value IRF5305 -> IRF5305 P-CH

Commit message: update and added uart menu
Connections:
- net N$13 renamed ADC0_POT
- net N$9 renamed ADC1_TEMP_SENS
- new net ADC2_BATT: IC1.25
- new net RESET: IC1.1
- new net XTAL1: IC1.9
- new net XTAL2: IC1.10
Changed lines of the file:
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@@
 <wire x1="15.875" y1="33.655" x2="15.875" y2="36.195" width="0.8128" layer="16"/>
 </signal>
-<signal name="N$9">
+<signal name="ADC1_TEMP_SENS">
 <contactref element="R7" pad="1"/>
 <contactref element="C7" pad="1"/>
@@
 <wire x1="29.21" y1="1.905" x2="29.21" y2="4.445" width="0.8128" layer="16"/>
 </signal>
-<signal name="N$13">
+<signal name="ADC0_POT">
 <contactref element="R8" pad="2"/>
 <contactref element="C8" pad="1"/>
@@
 <wire x1="61.2775" y1="18.415" x2="62.5475" y2="19.685" width="0.8128" layer="16"/>
 </signal>
+<signal name="ADC2_BATT">
+<contactref element="IC1" pad="25"/>
+</signal>
+<signal name="RESET">
+<contactref element="IC1" pad="1"/>
+</signal>
+<signal name="XTAL1">
+<contactref element="IC1" pad="9"/>
+</signal>
+<signal name="XTAL2">
+<contactref element="IC1" pad="10"/>
+</signal>
 </signals>
