File: hardware/eagle/rt_solder_simple_V1.2.sch (EAGLE design)
At the start: 33 parts, among them IC1 MEGA8-P, IC2 78L05, IC3 TLC27L2ACP, Q1 2N7000, Q3 IRF5305, X1 POWER, X2 Solder

Commit message: part list added
Parts:
- C1: value 4.7µF -> 4.7µF 10V
- C2, C5: value 470µF -> 470µF 16V
- L1: value 22µH -> 22µH or 10R
- Q1: value 2N7000 -> 2N7000 N-CH
- Q3: value IRF5305 -> IRF5305 P-CH

Commit message: update and added uart menu
Connections:
- net N$13 renamed ADC0_POT
- net N$9 renamed ADC1_TEMP_SENS
- new net ADC2_BATT: IC1.PC2(ADC2)
- new net RESET: IC1.PC6(/RESET)
- new net XTAL1: IC1.PB6(XTAL1/TOSC1)
- new net XTAL2: IC1.PB7(XTAL2/TOSC2)
Changed lines of the file:
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@@
 </segment>
 </net>
-<net name="N$9" class="0">
+<net name="ADC1_TEMP_SENS" class="0">
 <segment>
 <pinref part="R7" gate="G$1" pin="1"/>
@@
 <pinref part="IC1" gate="G$1" pin="PC1(ADC1)"/>
 <wire x1="144.78" y1="86.36" x2="116.84" y2="86.36" width="0.1524" layer="91"/>
+<label x="119.38" y="86.36" size="1.778" layer="95"/>
 </segment>
 </net>
@@
 </segment>
 </net>
-<net name="N$13" class="0">
+<net name="ADC0_POT" class="0">
 <segment>
 <pinref part="R8" gate="G$1" pin="2"/>
@@
 <wire x1="116.84" y1="88.9" x2="142.24" y2="88.9" width="0.1524" layer="91"/>
 <junction x="142.24" y="88.9"/>
+<label x="119.38" y="88.9" size="1.778" layer="95"/>
 </segment>
 </net>
@@
 <segment>
 <wire x1="38.1" y1="76.2" x2="38.1" y2="71.12" width="0.1524" layer="91"/>
-<wire x1="38.1" y1="71.12" x2="66.04" y2="71.12" width="0.1524" layer="91"/>
-<wire x1="66.04" y1="71.12" x2="66.04" y2="78.74" width="0.1524" layer="91"/>
+<wire x1="38.1" y1="71.12" x2="63.5" y2="71.12" width="0.1524" layer="91"/>
+<wire x1="63.5" y1="71.12" x2="63.5" y2="78.74" width="0.1524" layer="91"/>
 <pinref part="IC1" gate="G$1" pin="AVCC"/>
-<wire x1="66.04" y1="78.74" x2="68.58" y2="78.74" width="0.1524" layer="91"/>
+<wire x1="63.5" y1="78.74" x2="68.58" y2="78.74" width="0.1524" layer="91"/>
 <pinref part="C11" gate="G$1" pin="1"/>
 <junction x="38.1" y="71.12"/>
@@
 </segment>
 </net>
+<net name="ADC2_BATT" class="0">
+<segment>
+<pinref part="IC1" gate="G$1" pin="PC2(ADC2)"/>
+<wire x1="116.84" y1="83.82" x2="129.54" y2="83.82" width="0.1524" layer="91"/>
+<label x="119.38" y="83.82" size="1.778" layer="95"/>
+</segment>
+</net>
+<net name="RESET" class="0">
+<segment>
+<pinref part="IC1" gate="G$1" pin="PC6(/RESET)"/>
+<wire x1="68.58" y1="88.9" x2="53.34" y2="88.9" width="0.1524" layer="91"/>
+<label x="55.88" y="88.9" size="1.778" layer="95"/>
+</segment>
+</net>
+<net name="XTAL1" class="0">
+<segment>
+<pinref part="IC1" gate="G$1" pin="PB6(XTAL1/TOSC1)"/>
+<wire x1="68.58" y1="71.12" x2="66.04" y2="71.12" width="0.1524" layer="91"/>
+<wire x1="66.04" y1="71.12" x2="66.04" y2="68.58" width="0.1524" layer="91"/>
+<wire x1="66.04" y1="68.58" x2="55.88" y2="68.58" width="0.1524" layer="91"/>
+<label x="55.88" y="68.58" size="1.778" layer="95"/>
+</segment>
+</net>
+<net name="XTAL2" class="0">
+<segment>
+<pinref part="IC1" gate="G$1" pin="PB7(XTAL2/TOSC2)"/>
+<wire x1="68.58" y1="66.04" x2="55.88" y2="66.04" width="0.1524" layer="91"/>
+<label x="55.88" y="66.04" size="1.778" layer="95"/>
+</segment>
+</net>
